Commit message: Updated the rewards and cfg

File: IsaacLab_RFM/source/ext_loco/ext_loco/assets/SF_TRON1A_ARXR5ARM/assembly.urdf (robot description, URDF)
Before this commit: robot assembly, 19 links, 18 joints
Links:
- link eef_link: mass 0.0 -> 0.0001
Joints:
- joint gripper_fixed_joint: origin xyz=0.0999414 0.0000388 0.0767217 rpy=0 0.2618 0 -> xyz=0 0 0 rpy=0 0 0

Commit message: Sync training state and update R5 assets

File: IsaacLab_RFM/source/ext_loco/ext_loco/assets/SF_TRON1A_ARXR5ARM/assembly.urdf (robot description, URDF)
Before this commit: robot assembly, 19 links, 18 joints
Links:
- link base_link: geometry collision mesh filename=models/meshes/L5_umi/arm/base_link.STL; visual mesh filename=models/meshes/L5_umi/arm/base_link.STL
- link link1: mass 0.09728 -> 0.096804; geometry collision mesh filename=models/meshes/L5_umi/arm/link1.STL; visual mesh filename=models/meshes/L5_umi/arm/link1.STL
- link link2: mass 1.1477 -> 1.1988; geometry collision mesh filename=models/meshes/L5_umi/arm/link2.STL; visual mesh filename=models/meshes/L5_umi/arm/link2.STL
- link link3: mass 0.66 -> 0.84082; geometry collision mesh filename=models/meshes/L5_umi/arm/link3.STL; visual mesh filename=models/meshes/L5_umi/arm/link3.STL
- link link4: mass 0.11714 -> 0.12432; geometry collision mesh filename=models/meshes/L5_umi/arm/link4.STL; visual mesh filename=models/meshes/L5_umi/arm/link4.STL
- link link5: mass 0.6353 -> 0.63601; geometry collision mesh filename=models/meshes/L5_umi/arm/link5.STL; visual mesh filename=models/meshes/L5_umi/arm/link5.STL
- link link6: mass 0.902 -> 0.775
Joints:
- joint J3: origin xyz=-0.264 0 0 rpy=3.1416 0 0 -> xyz=-0.264 0 0 rpy=-3.1416 0 0
- joint J4: origin xyz=0.245 0 -0.06 rpy=0 0 0 -> xyz=0.245 -5E-05 -0.06 rpy=0 0 0
- joint J5: origin xyz=0.06775 -5E-05 -0.0865 rpy=0 0 0 -> xyz=0.073914 5E-05 -0.083391 rpy=0 0 0
- joint J6: origin xyz=0.02895 0 0.0865 rpy=3.1416 0 0 -> xyz=0.025286 0 0.083391 rpy=3.1416 0 0
- joint gripper_fixed_joint: origin xyz=0 0 0 rpy=0 0 0 -> xyz=0.15 0 0 rpy=0 0 0

File: IsaacLab_RFM/source/ext_loco/ext_loco/assets/SF_TRON1A_ARXR5ARM/models/L5_umi.urdf (robot description, URDF)
Before this commit: robot L5_umi, 9 links, 8 joints
Links:
- link base_link: geometry collision mesh filename=meshes/L5_umi/arm/base_link.STL; visual mesh filename=meshes/L5_umi/arm/base_link.STL
- link link1: mass 0.09728 -> 0.096804; geometry collision mesh filename=meshes/L5_umi/arm/link1.STL; visual mesh filename=meshes/L5_umi/arm/link1.STL
- link link2: mass 1.1477 -> 1.1988; geometry collision mesh filename=meshes/L5_umi/arm/link2.STL; visual mesh filename=meshes/L5_umi/arm/link2.STL
- link link3: mass 0.66 -> 0.84082; geometry collision mesh filename=meshes/L5_umi/arm/link3.STL; visual mesh filename=meshes/L5_umi/arm/link3.STL
- link link4: mass 0.11714 -> 0.12432; geometry collision mesh filename=meshes/L5_umi/arm/link4.STL; visual mesh filename=meshes/L5_umi/arm/link4.STL
- link link5: mass 0.6353 -> 0.63601; geometry collision mesh filename=meshes/L5_umi/arm/link5.STL; visual mesh filename=meshes/L5_umi/arm/link5.STL
- link link6: mass 0.902 -> 0.775
Joints:
- joint gripper_fixed_joint: origin xyz=0.0999414 0.0000388 0.0767217 rpy=0 0.2618 0 -> xyz=0.1039414 0.0000388 0.0767217 rpy=0 0.2618 0
- joint joint3: origin xyz=-0.264 0 0 rpy=3.1416 0 0 -> xyz=-0.264 0 0 rpy=-3.1416 0 0
- joint joint4: origin xyz=0.245 0 -0.06 rpy=0 0 0 -> xyz=0.245 -5E-05 -0.06 rpy=0 0 0
- joint joint5: origin xyz=0.06775 -5E-05 -0.0865 rpy=0 0 0 -> xyz=0.073914 5E-05 -0.083391 rpy=0 0 0
- joint joint6: origin xyz=0.02895 0 0.0865 rpy=3.1416 0 0 -> xyz=0.025286 0 0.083391 rpy=3.1416 0 0

File: IsaacLab_RFM/source/ext_loco/ext_loco/assets/SF_TRON1A_ARXR5ARM/models/X5.urdf (robot description, URDF)
Before this commit: robot X5, 8 links, 7 joints
Links:
- link base_link: geometry collision mesh filename=./meshes/X5/base_link.STL; visual mesh filename=./meshes/X5/base_link.STL

File: IsaacLab_RFM/source/ext_loco/ext_loco/assets/SF_TRON1A_ARXR5ARM/models/X5_no_gripper.urdf (robot description, URDF)
Before this commit: robot arx5_gopro, 8 links, 7 joints
Links:
- link base_link: geometry collision mesh filename=./meshes/X5/base_link.STL; visual mesh filename=./meshes/X5/base_link.STL
- link link1: geometry collision mesh filename=./meshes/X5/link1.STL; visual mesh filename=./meshes/X5/link1.STL
- link link2: geometry collision mesh filename=./meshes/X5/link2.STL; visual mesh filename=./meshes/X5/link2.STL
- link link3: geometry collision cylinder length=0.15 radius=0.02; visual mesh filename=./meshes/X5/link3.STL
- link link4: geometry collision cylinder length=0.05 radius=0.025; visual mesh filename=./meshes/X5/link4.STL
- link link5: geometry collision cylinder length=0.025 radius=0.02; visual mesh filename=./meshes/X5/link5.STL

Commit message: Update sim2sim control and SF TRON1 arm assets

File: IsaacLab_RFM/source/ext_loco/ext_loco/assets/SF_TRON1A_ARXR5ARM/assembly.urdf (robot description, URDF)
Before this commit: robot assembly, 19 links, 18 joints
Links:
- added link das_base_link, mass 0.0001
- link base_link: geometry collision mesh filename=models/meshes/L5_umi/arm/base_link.STL; visual mesh filename=models/meshes/L5_umi/arm/base_link.STL
- link link1: mass 0.09728 -> 0.096804; geometry collision mesh filename=models/meshes/L5_umi/arm/Link1.STL; visual mesh filename=models/meshes/L5_umi/arm/Link1.STL
- link link2: mass 1.1477 -> 1.1988; geometry collision mesh filename=models/meshes/L5_umi/arm/Link2.STL; visual mesh filename=models/meshes/L5_umi/arm/Link2.STL
- link link3: mass 0.66 -> 0.84082; geometry collision mesh filename=models/meshes/L5_umi/arm/Link3.STL; visual mesh filename=models/meshes/L5_umi/arm/Link3.STL
- link link4: mass 0.11714 -> 0.12432; geometry collision mesh filename=models/meshes/L5_umi/arm/Link4.STL; visual mesh filename=models/meshes/L5_umi/arm/Link4.STL
- link link5: mass 0.6353 -> 0.63601; geometry collision mesh filename=models/meshes/L5_umi/arm/Link5.STL; visual mesh filename=models/meshes/L5_umi/arm/Link5.STL
- link link6: mass 0.902 -> 0.775
Joints:
- added joint das_base_fixed_joint: type fixed, parent link6, child das_base_link, origin xyz=0.1039414 0.0000388 0.0767217 rpy=0 0.2618 0
- joint J3: origin xyz=-0.264 0 0 rpy=3.1416 0 0 -> xyz=-0.264 0 0 rpy=-3.1416 0 0
- joint J4: origin xyz=0.245 0 -0.06 rpy=0 0 0 -> xyz=0.245 -5E-05 -0.06 rpy=0 0 0
- joint J5: origin xyz=0.06775 -5E-05 -0.0865 rpy=0 0 0 -> xyz=0.073914 5E-05 -0.083391 rpy=0 0 0
- joint J6: origin xyz=0.02895 0 0.0865 rpy=3.1416 0 0 -> xyz=0.025286 0 0.083391 rpy=3.1416 0 0
- joint gripper_fixed_joint: origin xyz=0 0 0 rpy=0 0 0 -> xyz=0.15 0 0 rpy=0 0 0
